File: atmega328p.kicad_pcb (KiCad board)
At the start: 2 copper layers, 68.6 x 53.3 mm, 40 parts, among them CON1 Micro USB, CON2 AVR-ISP-6, IC1 DS3231M_SO16, IC2 LD1117, IC3 ATMEGA328P-TQFP32, M1 D1, P5 CONN_1, P6 CONN_1, P7 CONN_1, P8 CONN_1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

Commit message: Updated drill files
Parts:
- moved M1 0.16 mm to (123.0, 116.6)
Routing:
- net +3V3: track 134.0 -> 136.1 mm
Other:
- net class Default: clearance 0.2 -> 0.1; trace_width 0.4 -> 0.6
- rule trace_clearance: 0.2 -> 0.1
- rule trace_min: 0.4 -> 0.6

Commit message: minor changes and overall improvement
Connections:
- BATT1 pad 1: Net-(BATT1-Pad1) -> GND
- BATT1 pad 2: (no net) -> Net-(BATT1-Pad1)
- BATT1 pad 3: GND -> Net-(BATT1-Pad1)
Routing:
- net AREF: track 3.82 -> 48.8 mm, vias 0 -> 3
- net GND: track 309.7 -> 326.8 mm
- net Net-(BATT1-Pad1): track 29.1 -> 28.1 mm
Other:
- net class Default: trace_width 0.6 -> 0.4
- rule trace_min: 0.6 -> 0.4
- board text removed: "1"
